File: WT.sch (EAGLE design)
At the start: 115 parts, among them IC1 MC7805CDTG, IC2 NE5532D, IC3 NE5532D, IC4 QUAD_OPAMPD, IC5 LM4040B10, Q1 BSS123, Q2 SI2309CDS, Q3 BC846, SW3 SUB-MIN-SPDT, SW4 SUB-MIN-SPDT

Commit message: update board
Parts:
- removed LED1: MULTICOMP_703-1028, Rebel:MULTICOMP_703-1028
- removed Q3: BC846, transistor:BC846
- removed R44, R45: 510R, Rebel:R-EU_0603
- removed R48: 10k, Rebel:R-EU_0603
- removed R49: 1M, Rebel:R-EU_0603
- removed R50: 100k, Rebel:R-EU_0603
- removed SW3, SW4: SUB-MIN-SPDT, Rebel:SUB-MIN-SPDT
- removed TR: THONKICONN, Rebel:THONKICONN
- added D5, D6: BAT54S, diode:BAT54S
- added FM_L, FM_R: THONKICONN, Rebel:THONKICONN
- added IC6, IC7: LM1458D, linear:LM1458D
- added POTFM_L, POTFM_R, POTTUNE_L, POTTUNE_R: POT-ALPS-RK09L1140, Rebel:POT-ALPS-RK09L1140
- added R54, R59: 100k, Rebel:R-EU_0603
- added R56, R61: 33k, Rebel:R-EU_0603
- added R57, R62: 1k, Rebel:R-EU_0603
- added R58, R63: 100R, Rebel:R-EU_0603
- R36: value 1k -> 200k
- R43: value 510R -> 200k
- renumbered CV_A to CVX_L, CV_B to CVX_R, CV_C to CVY_L, CV_D to CVY_R, POT_A to POTX_L, POT_B to POTX_R, POT_C to POTY_L, POT_D to POTY_R
Connections:
- removed net GP10: SW4.O, TGP1-4.2
- removed net GP11: SW4.S, TGP1-4.1
- removed net GP1_LEDPWM: LGP1-5.1, R43.2
- removed net GP2_LEDPWM: LGP1-5.2, R44.2
- removed net GP5: LGP1-5.5, SW3.O
- removed net GP6_LEDPWM: LGP6-7.2, R45.2
- removed net GP7_TRIG: LGP6-7.1, Q3.C, R48.1
- removed net GP8: SW3.S, TGP1-4.5
- removed net GP9_CLK: R36.2, TGP1-4.4
- removed net N$37: Q3.B, R49.2, R50.2
- removed net N$38: R36.1, TR.4
- removed net N$40: LED1.CRED, R43.1
- removed net N$42: LED1.CGREEN, R45.1
- removed net N$43: LED1.CBLUE, R44.1
- removed net N$46: R50.1, TR.3
- new net ADC5: EXTSPI.4, R58.1
- new net ADC6: EXTSPI.3, R63.1
- new net ADC7: EXTSPI.2, POTTUNE_LG$1.2
- new net ADC8: EXTSPI.1, POTTUNE_RG$1.2
- new net N$45: POTFM_LG$1.2, R54.1
- new net N$47: IC6A.OUT, R56.2, R57.2
- new net N$48: D5.C1A2, R57.1, R58.2
- new net N$49: POTFM_RG$1.2, R59.1
- new net N$50: IC7B.-IN, R43.2, R59.2, R61.1
- new net N$51: FM_R.3, POTFM_RG$1.3
- new net N$52: IC7B.OUT, R61.2, R62.2
- new net N$53: D6.C1A2, R62.1, R63.2
- new net N$54: IC6A.-IN, R36.2, R54.2, R56.1
- new net N$57: FM_L.3, POTFM_LG$1.3
- net +3V3: now also D5.C2, D6.C2, POTTUNE_LG$1.1, POTTUNE_RG$1.1; no longer R48.2
- net +5V: no longer LED1.A
- net CV_REF: now also R36.1, R43.1
- net GND: now also D5.A1, D6.A1, FM_L.4, FM_L.5, FM_R.4, FM_R.5, IC6A.+IN, IC7B.+IN, POTFM_LG$1.1, POTFM_RG$1.1, POTTUNE_LG$1.3, POTTUNE_RG$1.3; no longer Q3.E, R49.1, SW3.P, SW4.P, TR.5
Other:
- moved on the sheet: C7, C8, IC2A, IC2B, R1, R10, R11, R12, R2, R3, R36, R4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
