File: WT.sch (EAGLE design)
At the start: 124 parts, among them IC1 MC7805CDTG, IC2 NE5532D, IC3 NE5532D, IC4 QUAD_OPAMPD, IC5 LM4040B10, IC6 TL072D, Q1 BSS123, Q2 SI2309CDS

Commit message: update final board
Changed lines of the file:
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@@
 <pinref part="C24" gate="G$1" pin="2"/>
 <wire x1="10.16" y1="238.76" x2="12.7" y2="238.76" width="0.1524" layer="91"/>
+<junction x="10.16" y="238.76"/>
 </segment>
 </net>
