File: WT.brd (EAGLE design)
At the start: 56 x 100 mm, 115 parts, among them IC1 MC7805CDTG, IC2 NE5532D, IC3 NE5532D, IC4 QUAD_OPAMPD, IC5 LM4040B10, Q1 BSS123, Q2 SI2309CDS, Q3 BC846, SW3 SUB-MIN-SPDT, SW4 SUB-MIN-SPDT

Commit message: update board
Parts:
- removed LED1: MULTICOMP_703-1028, Rebel:RGB-LED-703-1028
- removed Q3: BC846, transistor:SOT23
- removed R44, R45: 510R, Rebel:0603
- removed R48: 10k, Rebel:0603
- removed R49: 1M, Rebel:0603
- removed R50: 100k, Rebel:0603
- removed SW3, SW4: SUB-MIN-SPDT, Rebel:SUB-MIN-SPDT
- removed TR: THONKICONN, Rebel:THONKICONN
- added D5, D6: BAT54S, diode:SOT23
- added FM_L, FM_R: THONKICONN, Rebel:THONKICONN
- added IC6, IC7: LM1458D, linear:SO08
- added POTFM_L, POTFM_R, POTTUNE_L, POTTUNE_R: POT-ALPS-RK09L1140, Rebel:POT-ALPS-RK09L1140
- added R54, R59: 100k, Rebel:0603
- added R56, R61: 33k, Rebel:0603
- added R57, R62: 1k, Rebel:0603
- added R58, R63: 100R, Rebel:0603
- R36: value 1k -> 200k
- R43: value 510R -> 200k
- moved R43 358.8 mm to (-7.90, -264.8), flipped to the top, turned to 0 degrees
- moved R36 345.5 mm to (-7.90, -261.6), flipped to the top, turned to 0 degrees
- renumbered CV_A to CVX_L, CV_B to CVX_R, CV_C to CVY_L, CV_D to CVY_R, POT_A to POTX_L, POT_B to POTX_R, POT_C to POTY_L, POT_D to POTY_R
Connections:
- removed net GP10: SW4.1, TGP1-4.2
- removed net GP11: SW4.3, TGP1-4.1
- removed net GP1_LEDPWM: LGP1-5.1, R43.2
- removed net GP2_LEDPWM: LGP1-5.2, R44.2
- removed net GP5: LGP1-5.5, SW3.1
- removed net GP6_LEDPWM: LGP6-7.2, R45.2
- removed net GP7_TRIG: LGP6-7.1, Q3.3, R48.1
- removed net GP8: SW3.3, TGP1-4.5
- removed net GP9_CLK: R36.2, TGP1-4.4
- removed net N$37: Q3.1, R49.2, R50.2
- removed net N$38: R36.1, TR.P$2
- removed net N$40: LED1.P1, R43.1
- removed net N$42: LED1.P2, R45.1
- removed net N$43: LED1.P4, R44.1
- removed net N$46: R50.1, TR.P$3
- new net ADC5: EXTSPI.4, R58.1
- new net ADC6: EXTSPI.3, R63.1
- new net ADC7: EXTSPI.2, POTTUNE_L.2
- new net ADC8: EXTSPI.1, POTTUNE_R.2
- new net N$45: POTFM_L.2, R54.1
- new net N$47: IC6.1, R56.2, R57.2
- new net N$48: D5.3, R57.1, R58.2
- new net N$49: POTFM_R.2, R59.1
- new net N$50: IC7.6, R43.2, R59.2, R61.1
- new net N$51: FM_R.P$3, POTFM_R.3
- new net N$52: IC7.7, R61.2, R62.2
- new net N$53: D6.3, R62.1, R63.2
- new net N$54: IC6.2, R36.2, R54.2, R56.1
- new net N$57: FM_L.P$3, POTFM_L.3
- new net V+: IC6.8, IC7.8
- new net V-: IC6.4, IC7.4
- net +3V3: now also D5.2, D6.2, POTTUNE_L.1, POTTUNE_R.1; no longer R48.2
- net +5V: no longer LED1.P3
- net CV_REF: now also R36.1, R43.1
- net GND: now also D5.1, D6.1, FM_L.P$1, FM_L.P$2, FM_R.P$1, FM_R.P$2, IC6.3, IC7.5, POTFM_L.1, POTFM_R.1, POTTUNE_L.3, POTTUNE_R.3; no longer Q3.2, R49.1, SW3.2, SW4.2, TR.P$1
Routing:
- net N$46: track 112.0 -> 0.00 mm, vias 3 -> 0
- net GP8: track 98.9 -> 0.00 mm, vias 3 -> 0
- net GP5: track 74.9 -> 0.00 mm, vias 1 -> 0
- net N$38: track 68.0 -> 0.00 mm, vias 1 -> 0
- net GP10: track 54.4 -> 0.00 mm
- net GP11: track 45.0 -> 0.00 mm
- net N$42: track 31.0 -> 0.00 mm, vias 1 -> 0
- net N$43: track 29.9 -> 0.00 mm, vias 1 -> 0
- net N$40: track 26.8 -> 0.00 mm, vias 1 -> 0
- net +5V: track 133.5 -> 110.7 mm
- net GP9_CLK: track 10.5 -> 0.00 mm, vias 1 -> 0
- net GP7_TRIG: track 5.57 -> 0.00 mm
- net GP1_LEDPWM: track 5.03 -> 0.00 mm
- net GP2_LEDPWM: track 4.75 -> 0.00 mm
- net N$37: track 4.41 -> 0.00 mm
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
Commit message: update board
Parts:
- removed IC7: LM1458D, linear:SO08
- moved R43 351.2 mm to (33.4, 84.0), flipped to the bottom
- moved R36 350.8 mm to (36.4, 86.4), flipped to the bottom, turned to 90 degrees
- moved POTTUNE_R 302.2 mm to (42.2, 90.3)
- moved POTTUNE_L 236.0 mm to (13.6, 90.3)
- moved R62 225.7 mm to (27.0, 93.4), flipped to the bottom, turned to 180 degrees
- moved R63 225.4 mm to (24.4, 94.2), flipped to the bottom, turned to 270 degrees
- moved D6 197.6 mm to (22.5, 91.9), flipped to the bottom, turned to 90 degrees
- moved R59 188.3 mm to (26.7, 84.3), flipped to the bottom, turned to 180 degrees
- moved R61 188.3 mm to (29.8, 84.3), flipped to the bottom, turned to 180 degrees
- moved R56 162.6 mm to (26.8, 90.3), flipped to the bottom, turned to 270 degrees
- moved POTFM_R 159.5 mm to (42.2, 71.2)
- moved R57 158.6 mm to (26.8, 87.3), flipped to the bottom, turned to 90 degrees
- moved R58 157.4 mm to (25.2, 87.2), flipped to the bottom, turned to 270 degrees
- moved IC6 137.1 mm to (31.6, 87.9), flipped to the bottom, turned to 270 degrees
- moved R54 134.5 mm to (30.1, 91.4), flipped to the bottom
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Connections:
- net GND: now also IC6.2, IC6.6; no longer IC6.3, IC7.5
- net N$50: now also IC6.5; no longer IC7.6
- net N$52: now also IC6.7; no longer IC7.7
- net N$54: now also IC6.3; no longer IC6.2
- net V+: no longer IC7.8
- net V-: no longer IC7.4
Routing:
- net -12V: track 121.3 -> 213.6 mm
- net N$27: track 2.88 -> 60.4 mm
- net N$10: track 14.0 -> 64.0 mm
- net N$21: track 3.56 -> 46.9 mm
- net EXT_UART_RX: track 82.3 -> 46.3 mm
- net N$5: track 3.89 -> 36.0 mm
- net N$1: track 15.9 -> 44.7 mm
- net N$26: track 7.41 -> 35.5 mm
- net N$39: track 11.3 -> 36.9 mm
- net N$31: track 59.8 -> 83.9 mm
- net GP3_UART_TX: track 80.4 -> 57.9 mm
- net N$2: track 12.0 -> 33.8 mm
- net N$18: track 9.57 -> 31.3 mm
- net N$4: track 10.4 -> 31.7 mm
- net +5V: track 110.7 -> 89.6 mm
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