File: WT.brd (EAGLE design)
At the start: 56 x 100 mm, 124 parts, among them IC1 MC7805CDTG, IC2 NE5532D, IC3 NE5532D, IC4 QUAD_OPAMPD, IC5 LM4040B10, IC6 TL072D, Q1 BSS123, Q2 SI2309CDS

Commit message: update final board
Parts:
- moved C6 0.25 mm to (12.3, 14.5)
Routing:
- net GND: track 78.8 -> 19.7 mm
- net -12V: track 178.7 -> 179.6 mm

Commit message: update board
Parts:
- moved C2 16.4 mm to (24.4, 77.2)
- moved C13 1.27 mm to (30.5, 26.7)
- moved R17 1.27 mm to (33.0, 26.7)
- moved R18 1.27 mm to (24.1, 26.7)
- moved R19 1.27 mm to (21.6, 26.7)
- moved C10 0.76 mm to (30.5, 31.8)
- moved R14 0.76 mm to (24.1, 31.8)
Routing:
- net N$6: track 132.2 -> 109.6 mm
- net N$28: track 52.7 -> 30.3 mm
- net -12V: track 179.6 -> 166.0 mm
- net +12V: track 192.8 -> 181.5 mm
- net CV_REF: track 136.2 -> 144.6 mm
- net N$51: track 92.0 -> 95.7 mm
- net GP3_UART_TX: track 24.2 -> 27.8 mm
- net N$3: track 40.5 -> 37.6 mm
- net N$11: track 40.1 -> 42.4 mm
- net N$34: track 48.7 -> 50.9 mm
- net N$24: track 54.6 -> 56.7 mm
- net OUT_L: track 8.54 -> 10.7 mm
- net N$21: track 67.0 -> 69.1 mm
- net N$57: track 61.1 -> 63.1 mm
- net ADC3: track 9.68 -> 11.5 mm
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