File: WaveTable.sch (EAGLE design)
At the start: 122 parts, among them IC1 MC7805CDTG, IC2 NE5532D, IC3 NE5532D, IC4 QUAD_OPAMPD, IC5 LM4040B10, IC6 LM1458D, Q1 BSS123, Q2 SI2309CDS

Commit message: update board
Parts:
- removed LGP6-7: (no value), SparkFun:M02PTH
- removed POTFM_L, POTFM_R, POTTUNE_L, POTTUNE_R: POT-ALPS-RK09L1140, Rebel:POT-ALPS-RK09L1140
- removed R36, R43: 200k, Rebel:R-EU_0603
- added POT_D1, POT_D2: POT-ALPS-RK09L1140, Rebel:POT-ALPS-RK09L1140
- added R55, R66: 100k, Rebel:R-EU_0603
- added R65, R67: 33k, Rebel:R-EU_0603
- ADC: device SparkFun:M04PTH -> SparkFun:M06SIP
- renumbered POTX_L to POT_A, POTX_R to POT_B, POTY_L to POT_C, POTY_R to POT_D
Connections:
- removed net ADC7: EXTSPI.2, POTTUNE_LG$1.2
- removed net ADC8: EXTSPI.1, POTTUNE_RG$1.2
- new net N$55: IC6A.+IN, R55.2, R65.2
- new net N$56: IC6B.+IN, R66.2, R67.2
- net +3V3: no longer POTTUNE_LG$1.1, POTTUNE_RG$1.1
- net +5V: now also R55.1, R66.1
- net ADC1: now also ADC.6; no longer ADC.4
- net ADC2: now also ADC.5; no longer ADC.3
- net ADC3: now also ADC.4; no longer ADC.2
- net ADC4: now also ADC.3; no longer ADC.1
- net ADC5: now also ADC.2; no longer EXTSPI.4
- net ADC6: now also ADC.1; no longer EXTSPI.3
- net CV_REF: no longer R36.1, R43.1
- net GND: now also POT_D1G$1.1, POT_D2G$1.1, R65.1, R67.1; no longer IC6A.-IN, IC6B.-IN, POTFM_LG$1.1, POTFM_RG$1.1, POTTUNE_LG$1.3, POTTUNE_RG$1.3
- net N$45: now also POT_D1G$1.2; no longer POTFM_LG$1.2
- net N$49: now also POT_D2G$1.2; no longer POTFM_RG$1.2
- net N$50: now also IC6B.-IN; no longer IC6B.+IN, R43.2
- net N$51: now also POT_D2G$1.3; no longer POTFM_RG$1.3
- net N$54: now also IC6A.-IN; no longer IC6A.+IN, R36.2
- net N$57: now also POT_D1G$1.3; no longer POTFM_LG$1.3
Other:
- note added: "WaveTable"
- note removed: "Tesseract Rev03"
- moved on the sheet: C7, C8, D5, D6, FM_L, FM_R, IC2A, IC2B, IC6A, IC6B, R1, R10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
